File: payload/pcb/SAIL_OBC/SAIL_OBC.kicad_pcb (KiCad board)
At the start: 2 copper layers, 50.8 x 50.8 mm, 45 parts, among them J2 PPPC032LFBN-RC, J3 440055-6_6POS_2MM, J4 S4B-PH-K-S, J5 U.FL-R-SMT-1_10_, U1 RFM69HCW, U2 BNO055_SMT, U3 MICROSD-HRS_DM3D, U4 BMP390, U6 DEV-15583, Y1 CRYSTAL_32.768kHz

Commit message: Updated PCBs
Parts:
- removed the J4 at (114.1, 75.7)
- removed the U1 at (88.4, 57.0)
- added C7: 10nF, CustomFootprintLib:0805-NO (Capacitor), B.Cu at (111.8, 58.9)
- added J5: S5B-PH-K-S_LF__SN_, CustomFootprintLib:JST_S5B-PH-K-S_LF__SN_, F.Cu at (114.9, 75.7)
- added U7: RFM95W, CustomFootprintLib:RFMHCW_SMT, F.Cu at (88.4, 57.0)
- C1, C2: value 22 pF -> 22pF
- C3: value 0.1 uF -> 0.1uF
- C4: renamed from C5; value 1 uF -> 1uF
- C5: renamed from C8; value 22 pF -> 22pF
- C6: renamed from C7; value 100 nF -> 100nF
- C8: renamed from C9; value 10 uF -> 10uF
- J1: renamed from J3; value 440055-6_6POS_2MM -> 440055-6
- J4: renamed from J2; value PPPC032LFBN-RC -> PH2RA-06-UA
- R6: renamed from R9; value 40 -> 40.2
- TP1, TP2, TP3, TP4, TP5, TP6, TP7: footprint TestPoint:TestPoint_Pad_D1.0mm -> TestPoint:TestPoint_Pad_2.0x2.0mm
- U2: renamed from U5; value ~ -> W25Q64JVSSIQ
- moved TP3 1.02 mm to (112.0, 80.6)
- moved TP4 0.76 mm to (116.8, 80.6)
- moved C1 0.63 mm to (124.3, 49.3)
- moved C2 0.63 mm to (126.9, 49.3)
- moved TP7 0.13 mm to (89.2, 80.6)
- renumbered J5 to J3, R3 to R1, R8 to R10, R16 to R11, R15 to R12, R4 to R2, R12 to R3, R5 to R4, R6 to R5, R10 to R7, R11 to R8, R7 to R9, U3 to U1, U2 to U3, U6 to U5
Connections:
- U5 pad 9: unconnected-(U6-~9-Pad9) -> /GPS_EN
Routing:
- net /GPS_EN: track 0.00 -> 32.2 mm, vias 0 -> 2
- net /VOLTAGE: track 11.3 -> 15.2 mm
- net /TX: track 31.4 -> 32.1 mm
- net Net-(U3-XIN32): track 6.74 -> 6.10 mm
- net Net-(U3-XOUT32): track 8.20 -> 7.59 mm
- net /RX: track 31.1 -> 31.6 mm
Other:
- board text added: "01/2024"
- board text added: "EN"
- board text added: "SAIL OBC 1.0"
- board text removed: "SAIL 1.0 01/2024"
