File: payload/pcb/SAIL_OBC/SAIL_OBC.kicad_sch (KiCad schematic)
At the start: 45 parts, among them J1 440055-6_6POS_2MM, J2 S4B-PH-K-S, J3 U.FL-R-SMT-1_10_, J4 PPPC032LFBN-RC, U1 MICROSD-HRS_DM3D, U3 BNO055_SMT, U4 BMP390, U5 DEV-15583, U6 RFM69HCW, Y1 CRYSTAL_32.768kHz

Commit message: Updated PCBs
Parts:
- removed J2: S4B-PH-K-S, CustomFootprintLib:JST_S4B-PH-K-S_LF__SN_, symbol CustomComponents:S4B-PH-K-S_LF__SN_
- removed U6: RFM69HCW, CustomFootprintLib:RFMHCW_SMT, symbol CustomComponents:RFM69HCW_SMT
- added J5: S5B-PH-K-S_LF__SN_, CustomFootprintLib:JST_S5B-PH-K-S_LF__SN_, symbol CustomComponents:S5B-PH-K-S_LF__SN_
- added U7: RFM95W, CustomFootprintLib:RFMHCW_SMT, symbol CustomComponents:RFM69HCW_SMT
- BZ1: AVAILABILITY Unavailable -> (none); DESCRIPTION Buzzers Transducer, Externally Driven Piezo 3V 4kHz 60dB @ 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 -> (none); Distributor (none) -> DigiKey; Item # (none) -> 1; MAXIMUM_PACKAGE_HEIGHT 7.0mm -> (none); MF TDK -> (none); MP PS1240P02CT3 -> (none); Manufacturer (none) -> TDK Corporation; Mfg Part # (none) -> PS1240P02BT; PACKAGE SIP-5 TDK -> (none); PRICE None -> (none); Price (none) -> $0.63; Product URL (none) -> https://www.digikey.com/en/products/detail/tdk-corporation/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; Type (none) -> THT
- C1, C2, C5: Distributor (none) -> DigiKey; Item # (none) -> 2; Manufacturer (none) -> Samsung Electro-Mechanics; Mfg Part # (none) -> CL21C220JBANNNC; Package/Footprint (none) -> 0805; Price (none) -> $0.10; Product URL (none) -> https://www.digikey.com/en/products/detail/samsung-electro-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; Type (none) -> SMD
- C3: Distributor (none) -> DigiKey; Item # (none) -> 3; Manufacturer (none) -> YAGEO; Mfg Part # (none) -> CC0805KRX7R9BB104; Package/Footprint (none) -> 0805; Price (none) -> $0.10; Product URL (none) -> https://www.digikey.com/en/products/detail/yageo/CC0805KRX7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; Type (none) -> SMD
- C4: Distributor (none) -> DigiKey; Item # (none) -> 4; Manufacturer (none) -> Samsung Electro-Mechanics; Mfg Part # (none) -> CL21B105KBFNNNE; Package/Footprint (none) -> 0805; Price (none) -> $0.11; Product URL (none) -> https://www.digikey.com/en/products/detail/samsung-electro-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; Type (none) -> SMD
- C6: Distributor (none) -> DigiKey; Item # (none) -> 5; Manufacturer (none) -> YAGEO; Mfg Part # (none) -> CC0805KRX7R9BB104; Package/Footprint (none) -> 0805; Price (none) -> $0.10; Product URL (none) -> https://www.digikey.com/en/products/detail/yageo/CC0805KRX7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; Type (none) -> SMD
- C7: Distributor (none) -> DigiKey; Item # (none) -> 6; Manufacturer (none) -> Samsung Electro-Mechanics; Mfg Part # (none) -> CL21B103KBANNNC; Package/Footprint (none) -> 0805; Price (none) -> $0.10; Product URL (none) -> https://www.digikey.com/en/products/detail/samsung-electro-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; Type (none) -> SMD
- C8: Distributor (none) -> DigiKey; Item # (none) -> 7; Manufacturer (none) -> TDK Corporation; Mfg Part # (none) -> C2012X5R1V106K125AC; Package/Footprint (none) -> 0805; Price (none) -> $0.66; Product URL (none) -> https://www.digikey.com/en/products/detail/tdk-corporation/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; Type (none) -> SMD
- D1: Distributor (none) -> DigiKey; Item # (none) -> 8; Manufacturer (none) -> Adafruit; Mfg Part # (none) -> 159; Package/Footprint (none) -> 0805; Price (none) -> $2.00; Product URL (none) -> https://www.adafruit.com/product/159; Type (none) -> THT
- H1, H2, H3, H4: Item # (none) -> 9; Manufacturer (none) -> -; Mfg Part # (none) -> -; Notes (none) -> -; Package/Footprint (none) -> -; Price (none) -> -; Product URL (none) -> -; Type (none) -> -
- J1: value 440055-6_6POS_2MM -> 440055-6; Distributor (none) -> DigiKey; Item # (none) -> 10; MANUFACTURER TE -> (none); Manufacturer (none) -> TE Connectivity AMP Connectors; Mfg Part # (none) -> 440055-6; PARTREV R -> (none); Price (none) -> $0.41; Product URL (none) -> https://www.digikey.com/en/products/detail/te-connectivity-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; STANDARD Manufacturer Recommendations -> (none); Type (none) -> THT
- J3: AVAILABILITY Good -> (none); DESCRIPTION U.FL Series 6 Ghz 50 Ohm Ultra-small SMT Coaxial Cable Rece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 -> (none); Distributor (none) -> DigiKey; Item # (none) -> 11; MANUFACTURER Hirose -> (none); MP U.FL-R-SMT-1_10_ -> (none); Manufacturer (none) -> Hirose Electric Co Ltd; Mfg Part # (none) -> U.FL-R-SMT-1(10); PACKAGE None -> (none); PRICE 0.71 USD -> (none); Price (none) -> $1.35; Product URL (none) -> https://www.digikey.com/en/products/detail/hirose-electric-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; STANDARD Manufacturer Recommendation -> (none); Type (none) -> SMD
- J4: value PPPC032LFBN-RC -> PH2RA-06-UA; Item # (none) -> 12; Manufacturer (none) -> Adam Tech; Mfg Part # (none) -> PH2RA-06-UA; Price (none) -> $0.18; Product URL (none) -> https://www.digikey.com/en/products/detail/adam-tech/PH2RA-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; Type (none) -> THT
- JP1: Distributor (none) -> -; Item # (none) -> 14; Manufacturer (none) -> -; Mfg Part # (none) -> -; Notes (none) -> -; Package/Footprint (none) -> -; Price (none) -> -; Product URL (none) -> -; Type (none) -> -
- R1, R10, R11, R12, R2, R4, R5, R9: Distributor (none) -> DigiKey; Item # (none) -> 15; Manufacturer (none) -> Stackpole Electronics Inc; Mfg Part # (none) -> RMCF0805FT10K0; Package/Footprint (none) -> 0805; Price (none) -> $0.10; Product URL (none) -> https://www.digikey.com/en/products/detail/stackpole-electr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; Type (none) -> SMD
- R3: Distributor (none) -> DigiKey; Item # (none) -> 16; Manufacturer (none) -> Stackpole Electronics Inc; Mfg Part # (none) -> RMCF0805FT470R; Package/Footprint (none) -> 0805; Price (none) -> $0.10; Product URL (none) -> https://www.digikey.com/en/products/detail/stackpole-electr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; Type (none) -> SMD
- R6: value 40 -> 40.2; Distributor (none) -> DigiKey; Item # (none) -> 17; Manufacturer (none) -> Stackpole Electronics Inc; Mfg Part # (none) -> RMCF0805FT40R2; Package/Footprint (none) -> 0805; Price (none) -> $0.10; Product URL (none) -> https://www.digikey.com/en/products/detail/stackpole-electr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; Type (none) -> SMD
- R7, R8: Distributor (none) -> DigiKey; Item # (none) -> 18; Manufacturer (none) -> Stackpole Electronics Inc; Mfg Part # (none) -> RMCF0805FT1R00; Package/Footprint (none) -> 0805; Price (none) -> $0.10; Product URL (none) -> https://www.digikey.com/en/products/detail/stackpole-electr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; Type (none) -> SMD
- TP1, TP2, TP3, TP4: footprint TestPoint:TestPoint_Pad_D1.0mm -> TestPoint:TestPoint_Pad_2.0x2.0mm; Distributor (none) -> -; Item # (none) -> 19; Manufacturer (none) -> -; Mfg Part # (none) -> -; Notes (none) -> TestPoint; Package/Footprint (none) -> -; Price (none) -> -; Product URL (none) -> -
- TP5, TP6, TP7: footprint TestPoint:TestPoint_Pad_D1.0mm -> TestPoint:TestPoint_Pad_2.0x2.0mm; Distributor (none) -> -; Item # (none) -> 20; Manufacturer (none) -> -; Mfg Part # (none) -> -; Notes (none) -> TestPoint; Package/Footprint (none) -> -; Price (none) -> -; Product URL (none) -> -
- U1: Distributor (none) -> Mouser; Item # (none) -> 21; Manufacturer (none) -> Hirose Connector; Mfg Part # (none) -> DM3D-SF; Price (none) -> $1.82; Product URL (none) -> https://www.mouser.com/ProductDetail/Hirose-Connector/DM3D-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
- U2: value ~ -> W25Q64JVSSIQ; Distributor (none) -> DigiKey; Item # (none) -> 22; Manufacturer (none) -> Winbond Electronics; Mfg Part # (none) -> W25Q64JVSSIQ; Package/Footprint (none) -> 8-SOIC; Price (none) -> $1.03; Product URL (none) -> https://www.digikey.com/en/products/detail/winbond-electron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; Type (none) -> SMD
- U3: Distributor (none) -> DigiKey; Item # (none) -> 23; Manufacturer (none) -> Bosch Sensortec; Mfg Part # (none) -> BNO055; Package/Footprint (none) -> 28-TFLGA; Price (none) -> $15.37; Product URL (none) -> https://www.digikey.com/en/products/detail/bosch-sensortec/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; Type (none) -> SMD
- U4: Distributor (none) -> DigiKey; Item # (none) -> 24; Manufacturer (none) -> Bosch Sensortec; Mfg Part # (none) -> BMP390; Package/Footprint (none) -> 10-WFLGA; Price (none) -> $4.12; Product URL (none) -> https://www.digikey.com/en/products/detail/bosch-sensortec/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; Type (none) -> SMD
- U5: Availability In Stock -> (none); Check_prices https://www.snapeda.com/parts/DEV-15583/SparkFun+Electronic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 -> (none); Distributor (none) -> PJRC; Item # (none) -> 25; MANUFACTURER Sparkfun -> (none); MAXIMUM_PACKAGE_HEIGHT 5.87mm -> (none); MF SparkFun Electronics -> (none); MP DEV-15583 -> (none); Manufacturer (none) -> PJRC; Package None -> (none); Price None -> $23.80; Product URL (none) -> https://www.pjrc.com/store/teensy40.html; Purchase-URL https://www.snapeda.com/api/url_track_click_mouser/?unipart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 -> (none); STANDARD Manufacturer Recommendations -> (none); SnapEDA_Link https://www.snapeda.com/parts/DEV-15583/SparkFun+Electronic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 -> (none); Type (none) -> THT
- Y1: Distributor (none) -> DigiKey; Item # (none) -> 27; MANUFACTURER ECS Inc. -> (none); Manufacturer (none) -> ECS Inc.; Mfg Part # (none) -> ECS-.327-12.5-34B-TR; Package/Footprint (none) -> 2-SMD; Price (none) -> $0.44; Product URL (none) -> https://www.digikey.com/en/products/detail/ecs-inc/ECS-327-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; STANDARD Manufacturer recommendations -> (none); Type (none) -> SMD
Connections:
- net +3.3V: now also J5.1, U7.5 (VDD)
- net GND: now also J5.4, U7.16 (GND@3), U7.2 (GND@1), U7.9 (GND@2)
- net MISO: now also U7.10 (MISO)
- net MOSI: now also U7.11 (MOSI)
- net RADIO-CS: now also U7.13 (NSS)
- net RADIO_RST: now also U7.14 (RESET)
- net RX: now also J5.2
- net SCK: now also U7.12 (SCK)
- net TX: now also J5.3
- net at J3.1, JP1.1: now also U7.1 (ANT)
- net GPS_EN: now reaches U5.9 (~9)
- net GPS_EN: now also J5.5
- no-connect marks 27 -> 26
Other:
- note added: "01/17/2024"
- note added: "1.0"
- note added: "SAIL Onboard Computer"
