File: payload/pcb/SAIL_PDB/SAIL_PDB.kicad_pcb (KiCad board)
At the start: 4 copper layers, 50.8 x 50.8 mm, 48 parts, among them J1 440055-6_6POS_2MM, P1 TERMBLOCK_OSTTE020104_35MM, P2 TERMBLOCK_OSTTE020104_35MM, P3 TERMBLOCK_OSTTE020104_35MM, P4 TERMBLOCK_OSTTE020104_35MM, P5 TERMBLOCK_OSTTE020104_35MM, P6 TERMBLOCK_OSTTE020104_35MM, U1 DMN3051L-7, U2 AP63357_(SparkFun_Buck_Regula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, U3 DMN3051L-7, U4 AP63203

Commit message: Updated PCBs
Parts:
- removed D1, D2: CMD17-21VRD/TR8 LED, CustomFootprintLib:LED0805N_CML_(CMD17-21VRDTR8)
- removed the R12 at (105.2, 69.3)
- removed the R7 at (96.0, 57.0)
- removed the R8 at (106.4, 78.2)
- added R10: 3.9, Resistor_THT:R_Axial_DIN0204_L3.6mm_D1.6mm_P2.54mm_Vertical, F.Cu at (99.8, 75.7)
- C1, C6: value 10 uF -> 10uF
- C10: value 1 uF -> 1uF
- C2, C7: value 0.1 uF -> 0.1uF
- C3: value 4.7 pF -> 4.7pF
- C4, C5, C8, C9: value 22 uF -> 22uF
- L1: value 6.8 uH -> 6.8uH
- L2: value 4.7 uH -> 4.7uH
- P1: renamed from P4; value TERMBLOCK_OSTTE020104_35MM -> OSTTE020104
- P2: renamed from P1; value TERMBLOCK_OSTTE020104_35MM -> OSTTE020104
- P3: renamed from P2; value TERMBLOCK_OSTTE020104_35MM -> OSTTE020104
- P4: renamed from P3; value TERMBLOCK_OSTTE020104_35MM -> OSTTE020104
- P5, P6: value TERMBLOCK_OSTTE020104_35MM -> OSTTE020104
- R4: renamed from R5; value 157k -> 158k
- R6: renamed from R4; value 5.6 -> 2.7; footprint CustomFootprintLib:0805-NO-Resistor -> Resistor_THT:R_Axial_DIN0204_L3.6mm_D1.6mm_P2.54mm_Vertical
- R9: value 5.6 -> 470
- TP1, TP2, TP3, TP4: value TestPoint -> 5015; footprint TestPoint:TestPoint_THTPad_D1.5mm_Drill0.7mm -> CustomFootprintLib:KEYSTONE_5015_TEST
- moved R9 6.74 mm to (106.3, 78.0), turned to -90 degrees
- moved R6 2.62 mm to (83.9, 53.6)
- moved C3 2.03 mm to (101.6, 55.9)
- moved G*** 1.91 mm to (114.9, 62.9)
- moved R4 1.90 mm to (101.6, 57.8)
- moved C9 1.67 mm to (102.4, 68.2)
- moved C8 1.66 mm to (102.4, 70.2)
- moved C6 1.60 mm to (98.2, 67.3)
- moved C7 1.60 mm to (99.8, 62.1)
- moved L2 1.60 mm to (104.2, 63.8)
- moved U3 1.60 mm to (98.9, 64.8)
- moved R7 1.60 mm to (94.9, 67.6)
- moved R8 1.60 mm to (93.9, 64.5)
- moved R5 1.03 mm to (104.7, 54.9)
- moved R3 0.89 mm to (82.2, 60.5)
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- renumbered R2 to R1, R13 to R11, R14 to R12, R3 to R2, R1 to R3, R6 to R5, R10 to R7, R11 to R8, U2 to U1, U1 to U2, U4 to U3, U3 to U4
Connections:
- R9 pad 1: Net-(P5-Pad2) -> GND
- R9 pad 2: Net-(U3-DRAIN) -> /PYROCUT
- U4 pad TIP: Net-(U3-DRAIN) -> Net-(U4-DRAIN)
Routing:
- net +5V: track 43.4 -> 58.0 mm, vias 2 -> 3
- net /ARM: track 71.3 -> 84.7 mm
- net GND: track 13.6 -> 17.5 mm, vias 42 -> 39
- net Net-(P5-Pad2): track 30.4 -> 26.5 mm, vias 1 -> 0
- net Net-(U4-DRAIN): track 0.00 -> 3.40 mm
- net Net-(U3-DRAIN): track 2.72 -> 0.00 mm
- net Net-(D2-K): track 2.31 -> 0.00 mm
- net Net-(D1-K): track 2.23 -> 0.00 mm
- net /PY1: track 50.9 -> 49.5 mm
- net VCC: track 74.0 -> 74.7 mm, vias 5 -> 11
- added copper zone on B.Cu, net GND
- added copper zone on In1.Cu, net GND
- added copper zone on In2.Cu, net VCC
- removed copper zone on In1.Cu, net +5V
- removed copper zone on In2.Cu, net GND
Other:
- board text added: "01/2024"
- board text added: "Bridge R1/R8 to pull ENABLE High"
- board text added: "LANDING LEGS + -"
- board text added: "MASTER SWITCH"
- board text added: "MAX 25V"
- board text added: "Nichrome Wire"
- board text removed: "MAX 6S (22.2V)"
- board text removed: "PYRO + -"
- board text removed: "SWITCH"

Commit message: Updated pcb files
Parts:
- added JP1: Jumper_2_Open, Jumper:SolderJumper-2_P1.3mm_Open_Pad1.0x1.5mm, B.Cu at (87.7, 46.4)
- added JP3: Jumper_2_Open, Jumper:SolderJumper-2_P1.3mm_Open_Pad1.0x1.5mm, B.Cu at (85.6, 40.8)
- moved R1 0.25 mm to (94.7, 54.6)
- moved R2 0.18 mm to (97.6, 52.8)
- moved C5 0.05 mm to (98.2, 47.4)
Connections:
- P3 pad 1: VCC -> Net-(JP1-B)
Routing:
- net Net-(JP1-B): track 0.00 -> 12.6 mm
- net +5V: track 58.0 -> 67.8 mm, vias 3 -> 4
- net VCC: track 74.7 -> 67.0 mm
- net GND: track 17.5 -> 15.6 mm, vias 39 -> 36
- added copper zone on In2.Cu, net GND
Other:
- board text added: "Bridge R1/R7 to pull ENABLE High"
- board text added: "ONLY BRIDGE ONE FOR ARMING"
- board text added: "PYRO WIRE + -"
- board text added: "Voltage Divider"
- board text removed: "Bridge R1/R8 to pull ENABLE High"
- board text removed: "LANDING LEGS + -"
- board text removed: "Nichrome Wire"
