File: payload/pcb/SAIL_PDB/SAIL_PDB.kicad_sch (KiCad schematic)
At the start: 47 parts, among them J1 440055-6_6POS_2MM, P1 TERMBLOCK_OSTTE020104_35MM, P2 TERMBLOCK_OSTTE020104_35MM, P3 TERMBLOCK_OSTTE020104_35MM, P4 TERMBLOCK_OSTTE020104_35MM, P5 TERMBLOCK_OSTTE020104_35MM, P6 TERMBLOCK_OSTTE020104_35MM, U1 DMN3051L-7, U2 AP63357_(SparkFun_Buck_Regula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, U3 DMN3051L-7, U4 AP63203

Commit message: Updated PCBs
Parts:
- removed D1, D2: CMD17-21VRD/TR8 LED, CustomFootprintLib:LED0805N_CML_(CMD17-21VRDTR8), symbol Device:LED
- removed R2 (x2): 1k, CustomFootprintLib:0805-NO-Resistor, symbol Device:R
- removed R8: 470, CustomFootprintLib:0805-NO-Resistor, symbol Device:R
- removed TP1 (x4): TestPoint, TestPoint:TestPoint_THTPad_D1.5mm_Drill0.7mm, symbol Connector:TestPoint
- added R10: 3.9, Resistor_THT:R_Axial_DIN0204_L3.6mm_D1.6mm_P2.54mm_Vertical, symbol Device:R
- added TP1, TP2, TP3, TP4: 5015, CustomFootprintLib:KEYSTONE_5015_TEST, symbol CustomComponents:5011
- C1, C6: value 10 uF -> 10uF; Distributor (none) -> DigiKey; Item # (none) -> 1; MANUFACTURER (none) -> TDK Corporation; Mfg Part # (none) -> C2012X5R1V106K125AC; Package/Footprint (none) -> 0805; Price (none) -> $0.66; Produce Page (none) -> https://www.digikey.com/en/products/detail/tdk-corporation/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; Type (none) -> SMD
- C10: value 1 uF -> 1uF; Distributor (none) -> DigiKey; Item # (none) -> 5; MANUFACTURER (none) -> Samsung Electro-Mechanics; Mfg Part # (none) -> CL21B105KBFNNNE; Package/Footprint (none) -> 0805; Price (none) -> $0.11; Produce Page (none) -> https://www.digikey.com/en/products/detail/samsung-electro-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; Type (none) -> SMD
- C2, C7: value 0.1 uF -> 0.1uF; Distributor (none) -> DigiKey; Item # (none) -> 2; MANUFACTURER (none) -> YAGEO; Mfg Part # (none) -> CC0805KRX7R9BB104; Package/Footprint (none) -> 0805; Price (none) -> $0.10; Produce Page (none) -> https://www.digikey.com/en/products/detail/yageo/CC0805KRX7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; Type (none) -> SMD
- C3: value 4.7 pF -> 4.7pF; Distributor (none) -> DigiKey; Item # (none) -> 3; MANUFACTURER (none) -> KYOCERA AVX; Mfg Part # (none) -> KGM21BCG1H4R7BT; Package/Footprint (none) -> 0805; Price (none) -> $0.19; Produce Page (none) -> https://www.digikey.com/en/products/detail/kyocera-avx/KGM2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; Type (none) -> SMD
- C4, C5, C8, C9: value 22 uF -> 22uF; Distributor (none) -> DigiKey; Item # (none) -> 4; MANUFACTURER (none) -> TDK Corporation; Package/Footprint (none) -> 0805; Price (none) -> $0.82; Produce Page (none) -> https://www.digikey.com/en/products/detail/tdk-corporation/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; Type (none) -> SMD
- H1: Distributor (none) -> -; Item # (none) -> 7; MANUFACTURER (none) -> -; Mfg Part # (none) -> -; Notes (none) -> -; Package/Footprint (none) -> -; Produce Page (none) -> -
- H2, H3, H4: Distributor (none) -> -; Item # (none) -> 8; MANUFACTURER (none) -> -; Mfg Part # (none) -> -; Notes (none) -> -; Package/Footprint (none) -> -; Produce Page (none) -> -
- J1: Distributor (none) -> DigiKey; Item # (none) -> 9; MANUFACTURER TE -> TE Connectivity AMP Connectors; PARTREV R -> (none); Price (none) -> $0.41; Produce Page (none) -> https://www.digikey.com/en/products/detail/te-connectivity-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; STANDARD Manufacturer Recommendations -> (none); Type (none) -> SMD
- L1: value 6.8 uH -> 6.8uH; Distributor (none) -> DigiKey; Item # (none) -> 10; MANUFACTURER (none) -> TDK Corporation; Mfg Part # (none) -> VLS6045EX-6R8M; Price (none) -> $0.41; Produce Page (none) -> https://www.digikey.com/en/products/detail/tdk-corporation/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; Type (none) -> SMD
- L2: value 4.7 uH -> 4.7uH; Distributor (none) -> DigiKey; Item # (none) -> 11; MANUFACTURER (none) -> Taiyo Yuden; Mfg Part # (none) -> NRS4018T4R7MDGJ; Price (none) -> $0.23; Produce Page (none) -> https://www.digikey.com/en/products/detail/taiyo-yuden/NRS4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; Type (none) -> SMD
- P1: renamed from P4; value TERMBLOCK_OSTTE020104_35MM -> OSTTE020104; Distributor (none) -> DigiKey; Item # (none) -> 12; Mfg Part # (none) -> OSTTE020104; Price (none) -> $0.79; Produce Page (none) -> https://www.digikey.com/en/products/detail/on-shore-technol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; Type (none) -> THT
- P2: renamed from P1; value TERMBLOCK_OSTTE020104_35MM -> OSTTE020104; Distributor (none) -> DigiKey; Item # (none) -> 12; Mfg Part # (none) -> OSTTE020104; Price (none) -> $0.79; Produce Page (none) -> https://www.digikey.com/en/products/detail/on-shore-technol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; Type (none) -> THT
- P3: renamed from P2; value TERMBLOCK_OSTTE020104_35MM -> OSTTE020104; Distributor (none) -> DigiKey; Item # (none) -> 12; Mfg Part # (none) -> OSTTE020104; Price (none) -> $0.79; Produce Page (none) -> https://www.digikey.com/en/products/detail/on-shore-technol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; Type (none) -> THT
- P4: renamed from P3; value TERMBLOCK_OSTTE020104_35MM -> OSTTE020104; Distributor (none) -> DigiKey; Item # (none) -> 12; Mfg Part # (none) -> OSTTE020104; Price (none) -> $0.79; Produce Page (none) -> https://www.digikey.com/en/products/detail/on-shore-technol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; Type (none) -> THT
- P5, P6: value TERMBLOCK_OSTTE020104_35MM -> OSTTE020104; Distributor (none) -> DigiKey; Item # (none) -> 12; Mfg Part # (none) -> OSTTE020104; Price (none) -> $0.79; Produce Page (none) -> https://www.digikey.com/en/products/detail/on-shore-technol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; Type (none) -> THT
- R1: Distributor (none) -> DigiKey; Item # (none) -> 20; MANUFACTURER (none) -> Stackpole Electronics Inc; Mfg Part # (none) -> RMCF0805FT3K90; Package/Footprint (none) -> 0805; Price (none) -> $0.10; Produce Page (none) -> https://www.digikey.com/en/products/detail/stackpole-electr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; Type (none) -> SMD
- R2: Distributor (none) -> DigiKey; Item # (none) -> 14; MANUFACTURER (none) -> Stackpole Electronics Inc; Mfg Part # (none) -> RMCF0805FT3K60; Package/Footprint (none) -> 0805; Price (none) -> $0.10; Produce Page (none) -> https://www.digikey.com/en/products/detail/stackpole-electr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; Type (none) -> SMD
- R2: Distributor (none) -> DigiKey; Item # (none) -> 15; MANUFACTURER (none) -> Stackpole Electronics Inc; Mfg Part # (none) -> RMCF0805FT470R; Package/Footprint (none) -> 0805; Price (none) -> $0.10; Produce Page (none) -> https://www.digikey.com/en/products/detail/stackpole-electr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; Type (none) -> SMD
- R2: Distributor (none) -> DigiKey; Item # (none) -> 13; MANUFACTURER (none) -> KOA Speer Electronics, Inc.; Mfg Part # (none) -> RK73B2ATTD683J; Package/Footprint (none) -> 0805; Price (none) -> $0.10; Produce Page (none) -> https://www.digikey.com/en/products/detail/koa-speer-electr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; Type (none) -> SMD
- R2: Distributor (none) -> DigiKey; Item # (none) -> 17; MANUFACTURER (none) -> Stackpole Electronics Inc; Mfg Part # (none) -> RMCF0805FT30K0; Package/Footprint (none) -> 0805; Price (none) -> $0.10; Produce Page (none) -> https://www.digikey.com/en/products/detail/stackpole-electr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; Type (none) -> SMD
- R2: value 157k -> 158k; Distributor (none) -> DigiKey; Item # (none) -> 16; MANUFACTURER (none) -> YAGEO; Mfg Part # (none) -> RC0805FR-07158KL; Package/Footprint (none) -> 0805; Price (none) -> $0.10; Produce Page (none) -> https://www.digikey.com/en/products/detail/yageo/RC0805FR-0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; Type (none) -> SMD
- R3: renamed from R1; Distributor (none) -> DigiKey; Item # (none) -> 15; MANUFACTURER (none) -> Stackpole Electronics Inc; Mfg Part # (none) -> RMCF0805FT470R; Package/Footprint (none) -> 0805; Price (none) -> $0.10; Produce Page (none) -> https://www.digikey.com/en/products/detail/stackpole-electr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; Type (none) -> SMD
- R6: renamed from R4; value 5.6 -> 2.7; footprint CustomFootprintLib:0805-NO-Resistor -> Resistor_THT:R_Axial_DIN0204_L3.6mm_D1.6mm_P2.54mm_Vertical; Distributor (none) -> DigiKey; Item # (none) -> 18; MANUFACTURER (none) -> Stackpole Electronics Inc; Mfg Part # (none) -> RMCF0805FT5R60; Package/Footprint (none) -> 0805; Price (none) -> $0.10; Produce Page (none) -> https://www.digikey.com/en/products/detail/stackpole-electr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; Type (none) -> SMD
- R9: value 5.6 -> 470; Distributor (none) -> DigiKey; Item # (none) -> 15; MANUFACTURER (none) -> Stackpole Electronics Inc; Mfg Part # (none) -> RMCF0805FT470R; Package/Footprint (none) -> 0805; Price (none) -> $0.10; Produce Page (none) -> https://www.digikey.com/en/products/detail/stackpole-electr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; Type (none) -> SMD
- U1: renamed from U2; Distributor (none) -> DigiKey; Item # (none) -> 22; MANUFACTURER (none) -> Diodes Incorporated; Mfg Part # (none) -> AP63357DV-7; Package/Footprint (none) -> 13-PowerVFDFN; Price (none) -> $0.94; Produce Page (none) -> https://www.digikey.com/en/products/detail/diodes-incorpora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; Type (none) -> SMD
- U2: renamed from U1; Distributor (none) -> DigiKey; Item # (none) -> 24; MANUFACTURER (none) -> Diodes Incorporated; Mfg Part # (none) -> DMN3051L-7; Package/Footprint (none) -> SOT-23-3; Price (none) -> $0.46; Produce Page (none) -> https://www.digikey.com/en/products/detail/diodes-incorpora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; Type (none) -> SMD
- U3: renamed from U4; Distributor (none) -> DigiKey; Item # (none) -> 23; MANUFACTURER (none) -> Diodes Incorporated; Mfg Part # (none) -> AP63203WU-7; Package/Footprint (none) -> TSOT-23-6; Price (none) -> $0.87; Produce Page (none) -> https://www.digikey.com/en/products/detail/diodes-incorpora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; Type (none) -> SMD
- U4: renamed from U3; Distributor (none) -> DigiKey; Item # (none) -> 24; MANUFACTURER (none) -> Diodes Incorporated; Mfg Part # (none) -> DMN3051L-7; Package/Footprint (none) -> SOT-23-3; Price (none) -> $0.46; Produce Page (none) -> https://www.digikey.com/en/products/detail/diodes-incorpora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; Type (none) -> SMD
Connections:
- net +3.3V: now also TP3.TP
- net +5V: now also TP2.TP
- net GND: now also R9.1, TP4.TP
- net PYROCUT: now also R9.2
- net VCC: now also TP1.TP
- net at P5.2, P6.2: now also R10.2; no longer R9.1
- net at U4.TIP (DRAIN): now also R10.1; no longer R9.2
Other:
- note added: "01/17/2024"
- note added: "1.0"
- note added: "36g nichrome wire 26Ohm/ft -> 2-3in. 4.34-6.5Ohm"
- note added: "Arm Switch"
- note added: "Battery"
- note added: "Landing Leg Release"
- note added: "PWR Switch"
- note added: "R10/R12 Values 7.2V-9.6V -> 3.9 Ohm / 2 -> 0.92A-1.23A 21.6 - 25.2V -> 11Ohm / 2 -> 0.98A - 1.15A"
- note added: "R6 Values 9V -> 6.5 + 2.7Ohm -> 0.98A 25.2V -> 6.5 + 20Ohm -> 0.95A"
- note added: "SAIL Power Distribution Board"
- note removed: "4.0 A Id"
- note removed: "Battery Input / Switch / Pyro Control"
- note removed: "OUTDATED: 1/5 sufficient up to 4S (14.8V)"
- note removed: "R4 Values 9V -> 5.6Ohm -> 1.6A 25.2V -> 16Ohm -> 1.58A"
- note removed: "R9 Values 9V -> 3.9Ohm -> 2.3A / 2 = 1.15A each 25.2V -> 10Ohm -> 2.52A / 2 = 1.26A each"
- note removed: "change to CMD17-21VRC/TR8 varying voltage source? good idea for led?"
- note removed: "unsure if current is high enough to break rubber band"
- moved on the sheet: P1, P2, P3, P4, P5, P6, R3, R6, U2, U4

Commit message: Updated pcb files
Parts:
- added JP1, JP3: Jumper_2_Open, Jumper:SolderJumper-2_P1.3mm_Open_Pad1.0x1.5mm, symbol Jumper:Jumper_2_Open
Connections:
- net +5V: now also JP1.1 (A)
- net VCC: now also JP3.1 (A); no longer P3.1
- new net: JP1.2 (B), JP3.2 (B), P3.1
- no-connect marks 3 -> 2
Other:
- note added: "25.2V LiPo Battery UVLO Hi: 21.9V UVLO Lo: 21.6V (6*3.6) R1 = 68k, R2 = 3.6k Refer to datasheet for R1/R2 equation"
- note added: "25.2V LiPo Battery UVLO Hi: 21.9V UVLO Lo: 21.6V (6*3.6) R7 = 68k, R8 = 3.6k Refer to datasheet for R7/R8"
- note added: "3.3V = 2^10-1 = 1023 and 1/10 voltage divider gives 1023 / (3.3 x 10) = 31 Code: Voltage=(float)analogRead(pin#)/31;"
- note added: "9V Li-Ion Battery UVLO Hi: 6.6V UVLO Lo: 6.4V R1 = 43k, R2 = 8.2k Refer to datasheet for R1/R2"
- note added: "9V Li-Ion Battery UVLO Hi: 6.6V UVLO Lo: 6.4V R1 = 43k, R2 = 8.2k Refer to datasheet for R7/R8"
- note added: "If we need Buck +5V output to fire charges"
- note removed: "3.3V = 2^10-1 = 1023 and 1/5 voltage divider gives 1023 / (3.3 x 5) = 62 Code: Voltage=(float)analogRead(15)/62;"
- note removed: "UVLO Hi: 21.9V UVLO Lo: 21.6V (6*3.6) Refer to datasheet for R10/R11"
- note removed: "UVLO Hi: 21.9V UVLO Lo: 21.6V (6*3.6) Refer to datasheet for R2/R3"
- moved on the sheet: C10, P3, R1, R2

Commit message: Updated PCBs
im dumb
Parts:
- C1, C6: Distributor Part Number (none) -> 445-14418-1-ND
- C10: Distributor Part Number (none) -> 1276-1029-1-ND
- C2, C7: Distributor Part Number (none) -> 311-1140-1-ND
- C3: Distributor Part Number (none) -> 478-KGM21BCG1H4R7BTCT-ND
- C4, C5, C8, C9: Distributor Part Number (none) -> 445-14428-1-ND
- H1, H2, H3, H4: Distributor Part Number (none) -> -; Price (none) -> -; Type (none) -> -
- J1: Distributor Part Number (none) -> A100047-ND
- JP1, JP3: Distributor (none) -> -; Distributor Part Number (none) -> -; Item # (none) -> 10; MANUFACTURER (none) -> -; Mfg Part # (none) -> -; Notes (none) -> -; Package/Footprint (none) -> -; Price (none) -> -; Produce Page (none) -> -; Type (none) -> -
- L1: Distributor Part Number (none) -> 445-173057-1-ND; Item # 10 -> 11
- L2: Distributor Part Number (none) -> 587-2893-1-ND; Item # 11 -> 12
- P1, P2, P3, P4, P5, P6: Distributor Part Number (none) -> ED2740-ND; Item # 12 -> 13
- R1: Distributor Part Number (none) -> RMCF0805FT3K90CT-ND; Item # 20 -> 21
- R10: Distributor Part Number (none) -> PPC3.9W-1CT-ND; Item # 15 -> 20; MANUFACTURER Stackpole Electronics Inc -> (none); Mfg Part # RMCF0805FT470R -> (none); Produce Page https://www.digikey.com/en/products/detail/stackpole-electr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 -> https://www.digikey.com/en/products/detail/vishay-beyschlag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; Type SMD -> THT
- R2: Distributor Part Number (none) -> RMCF0805FT3K60CT-ND; Item # 14 -> 15
- R2, R3, R9: Distributor Part Number (none) -> RMCF0805FT470RCT-ND; Item # 15 -> 16
- R2: Distributor Part Number (none) -> 2019-RK73B2ATTD683JCT-ND; Item # 13 -> 14
- R2: Distributor Part Number (none) -> RMCF0805FT30K0CT-ND; Item # 17 -> 18
- R2: Distributor Part Number (none) -> 311-158KCRCT-ND; Item # 16 -> 17
- R6: Distributor Part Number (none) -> S2.7HCT-ND; Item # 18 -> 15; MANUFACTURER Stackpole Electronics Inc -> (none); Mfg Part # RMCF0805FT5R60 -> (none); Produce Page https://www.digikey.com/en/products/detail/stackpole-electronics-inc/RMCF0805FT5R60/1713196 -> https://www.digikey.com/en/products/detail/stackpole-electronics-inc/CFM12JT2R70/1741892; Type SMD -> THT
- TP1, TP2, TP3, TP4: Distributor (none) -> DigiKey; Distributor Part Number (none) -> 36-5015CT-ND; Item # (none) -> 22; MANUFACTURER (none) -> Keystone Electronics; Mfg Part # (none) -> 5015; Price (none) -> $0.45; Produce Page (none) -> https://www.digikey.com/en/products/detail/keystone-electro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; Type (none) -> SMD
- U1: Distributor Part Number (none) -> 31-AP63357DV-7CT-ND; Item # 22 -> 23
- U2, U4: Distributor Part Number (none) -> DMN3051LDICT-ND
- U3: Distributor Part Number (none) -> AP63203WU-7DICT-ND; Item # 23 -> 25
Other:
- moved on the sheet: JP1, JP3, P3
